File: jlc_board/reptile-monitor-s2.kicad_sch (KiCad schematic)
At the start: 49 parts, among them J1 USB_C_Receptacle_USB2.0, J2 AC_IN, J3 Conn_01x08, J7 LOAD0, J8 LOAD1, K1 1462041-7, K2 1462041-7, SW1 RESET, SW2 BOOT, U1 ESP32-S2-WROVER, U2 TPS2112PW, U3 AP2112K-3.3, U4 MDC3105LT1G, U5 MDC3105LT1G, Y1 32.768KHz 12.5p

Commit message: rev2
Parts:
- removed K1, K2: 1462041-7, Reptile_Monitor:TE_Connectivity-1462041-7-0-0, symbol Reptile_Monitor:1462041-7
- removed TP2: SRC, TestPoint:TestPoint_THTPad_1.0x1.0mm_Drill0.5mm, symbol Connector:TestPoint_Probe
- removed TP4: 5V, TestPoint:TestPoint_THTPad_1.0x1.0mm_Drill0.5mm, symbol Connector:TestPoint_Probe
- removed TP5: VCC, TestPoint:TestPoint_THTPad_1.0x1.0mm_Drill0.5mm, symbol Connector:TestPoint_Probe
- removed TP6: VBUS, TestPoint:TestPoint_THTPad_1.0x1.0mm_Drill0.5mm, symbol Connector:TestPoint_Probe
- added K1, K2: ALDP105W, reptile-monitor:Panasonic-ALDP105W-Manufacturer_Recommended, symbol Reptile_Monitor:ALDP105W
- J2: footprint Connector_Molex:Molex_Micro-Fit_3.0_43650-0215_1x02_P3.00mm_Vertical -> reptile-monitor:Molex-43650-0215-0-0-MFG; symbol Connector_Generic:Conn_01x02 -> Reptile_Monitor:43650-0215; 3DS Part Number (none) -> 610-00029; category (none) -> Conn; contact material (none) -> Tin,Brass; current rating (none) -> 8.5A; device class L1 (none) -> Connectors; device class L2 (none) -> Board to Board Connectors; device class L3 (none) -> unset; digikey description (none) -> CONN HEADER 2POS 3MM VERT TIN; digikey part number (none) -> WM1917-ND; footprint url (none) -> http://www.molex.com/pdm_docs/sd/436500200_sd.pdf; height (none) -> 10.15mm; is connector (none) -> yes; is male (none) -> yes; lead free (none) -> yes; library id (none) -> bd6a551cc925a413; manufacturer (none) -> Molex; mouser description (none) -> Headers & Wire Housings MICRO-FIT 3.0 HEADER; mouser part number (none) -> 538-43650-0215; number of contacts (none) -> 2; number of rows (none) -> 1; package (none) -> CONN_2POS; rohs (none) -> yes; temperature range high (none) -> +105°C; temperature range low (none) -> -40°C; voltage rating (none) -> 600V
- J7: value LOAD0 -> LOAD1; footprint Connector_Molex:Molex_Micro-Fit_3.0_43650-0215_1x02_P3.00mm_Vertical -> reptile-monitor:Molex-43650-0215-0-0-MFG; symbol Connector_Generic:Conn_01x02 -> Reptile_Monitor:43650-0215; 3DS Part Number (none) -> 610-00029; category (none) -> Conn; contact material (none) -> Tin,Brass; current rating (none) -> 8.5A; device class L1 (none) -> Connectors; device class L2 (none) -> Board to Board Connectors; device class L3 (none) -> unset; digikey description (none) -> CONN HEADER 2POS 3MM VERT TIN; digikey part number (none) -> WM1917-ND; footprint url (none) -> http://www.molex.com/pdm_docs/sd/436500200_sd.pdf; height (none) -> 10.15mm; is connector (none) -> yes; is male (none) -> yes; lead free (none) -> yes; library id (none) -> bd6a551cc925a413; manufacturer (none) -> Molex; mouser description (none) -> Headers & Wire Housings MICRO-FIT 3.0 HEADER; mouser part number (none) -> 538-43650-0215; number of contacts (none) -> 2; number of rows (none) -> 1; package (none) -> CONN_2POS; rohs (none) -> yes; temperature range high (none) -> +105°C; temperature range low (none) -> -40°C; voltage rating (none) -> 600V
- J8: value LOAD1 -> LOAD2; footprint Connector_Molex:Molex_Micro-Fit_3.0_43650-0215_1x02_P3.00mm_Vertical -> reptile-monitor:Molex-43650-0215-0-0-MFG; symbol Connector_Generic:Conn_01x02 -> Reptile_Monitor:43650-0215; 3DS Part Number (none) -> 610-00029; category (none) -> Conn; contact material (none) -> Tin,Brass; current rating (none) -> 8.5A; device class L1 (none) -> Connectors; device class L2 (none) -> Board to Board Connectors; device class L3 (none) -> unset; digikey description (none) -> CONN HEADER 2POS 3MM VERT TIN; digikey part number (none) -> WM1917-ND; footprint url (none) -> http://www.molex.com/pdm_docs/sd/436500200_sd.pdf; height (none) -> 10.15mm; is connector (none) -> yes; is male (none) -> yes; lead free (none) -> yes; library id (none) -> bd6a551cc925a413; manufacturer (none) -> Molex; mouser description (none) -> Headers & Wire Housings MICRO-FIT 3.0 HEADER; mouser part number (none) -> 538-43650-0215; number of contacts (none) -> 2; number of rows (none) -> 1; package (none) -> CONN_2POS; rohs (none) -> yes; temperature range high (none) -> +105°C; temperature range low (none) -> -40°C; voltage rating (none) -> 600V
- R10: value 10K -> 10k
- R9: value 500R -> 500r
- SW1: value RESET -> RST; footprint Reptile_Monitor:Alps_SKRK -> reptile-monitor:Omron-B3U-1000P-MFG; symbol Switch:SW_Push -> Reptile_Monitor:B3U-1000P; ambient temperature range high (none) -> +70°C; ambient temperature range low (none) -> -25°C; automotive (none) -> No; category (none) -> Switch; contact current rating (none) -> 50mA; contact resistance (none) -> 100mΩ; current rating (none) -> 0.05A; device class L1 (none) -> Electromechanical; device class L2 (none) -> Switches; device class L3 (none) -> Tactile Switches; digikey description (none) -> SWITCH TACTILE SPST-NO 0.05A 12V; digikey part number (none) -> SW1020CT-ND; electromechanical life (none) -> 200000Cycles; height (none) -> 1.75mm; lead free (none) -> Yes; library id (none) -> b933800f68cdf4c7; manufacturer (none) -> Omron; mount (none) -> Surface Mount; mouser part number (none) -> 653-B3U-1000P; operating force (none) -> 1.5N; package (none) -> SW_SMT_3MM2_2MM7; rohs (none) -> Yes; temperature range high (none) -> +70°C; temperature range low (none) -> -25°C; throw configuration (none) -> SPST-NO; voltage rating DC (none) -> 12V
- SW2: footprint Reptile_Monitor:Alps_SKRK -> reptile-monitor:Omron-B3U-1000P-MFG; symbol Switch:SW_Push -> Reptile_Monitor:B3U-1000P; ambient temperature range high (none) -> +70°C; ambient temperature range low (none) -> -25°C; automotive (none) -> No; category (none) -> Switch; contact current rating (none) -> 50mA; contact resistance (none) -> 100mΩ; current rating (none) -> 0.05A; device class L1 (none) -> Electromechanical; device class L2 (none) -> Switches; device class L3 (none) -> Tactile Switches; digikey description (none) -> SWITCH TACTILE SPST-NO 0.05A 12V; digikey part number (none) -> SW1020CT-ND; electromechanical life (none) -> 200000Cycles; height (none) -> 1.75mm; lead free (none) -> Yes; library id (none) -> b933800f68cdf4c7; manufacturer (none) -> Omron; mount (none) -> Surface Mount; mouser part number (none) -> 653-B3U-1000P; operating force (none) -> 1.5N; package (none) -> SW_SMT_3MM2_2MM7; rohs (none) -> Yes; temperature range high (none) -> +70°C; temperature range low (none) -> -25°C; throw configuration (none) -> SPST-NO; voltage rating DC (none) -> 12V
- U3: footprint Package_TO_SOT_SMD:SOT-23-5 -> SamacSys_Parts:SOIC127P600X170-8N; symbol Regulator_Linear:AP2112K-3.3 -> SamacSys_Parts:AP2112M-3.3TRG1; Height (none) -> 1.7; Manufacturer_Name (none) -> Diodes Inc.; Manufacturer_Part_Number (none) -> AP2112M-3.3TRG1; Mouser Part Number (none) -> 621-AP2112M-3.3TRG1; Mouser Price/Stock (none) -> https://www.mouser.co.uk/ProductDetail/Diodes-Incorporated/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
Connections:
- net +3V3: now also U3.1 (VOUT); no longer U3.5 (VOUT)
- net +5V: now also R12.2, U3.8 (VIN), K1.1, K2.1; no longer R12.1, U3.1 (VIN)
- net AC_L: now also K1.3 (COM), K2.3 (COM)
- net EN: now also SW1.1; no longer SW1.2
- net GND: now also SW1.2, SW2.2, U3.6 (GND_1), U3.7 (GND_2); no longer SW1.1, SW2.1, U3.2 (GND)
- net IO0: now also SW2.1; no longer SW2.2
- net IO17: now also U4.1 (Vin); no longer U5.1 (Vin)
- net IO18: now also U5.1 (Vin); no longer U4.1 (Vin)
- net at U5.3 (Vout): now also K2.4
- net at U3.3 (NC_2): no longer R12.2
- net at U4.3 (Vout): now also K1.4
- net LOAD_0 renamed LOAD1
- net LOAD1: now also K1.2 (NO)
- net LOAD_1 renamed LOAD2
- net LOAD2: now also K2.2 (NO)
- new net: R12.1, U3.5 (EN)
- no-connect marks 2 -> 5
Other:
- moved on the sheet: D2, R12, R13, U5

Commit message: rev 2
Connections:
- net GND: no longer J1.S1 (SHIELD)
- no-connect marks 5 -> 6
Changed lines of the file:
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@@
 (kicad_sch (version 20210406) (generator eeschema)
   (paper "A4")
-  (junction (at 26.67 66.675) (diameter 0.9144) (color 0 0 0 0))
   (junction (at 36.83 104.14) (diameter 0.9144) (color 0 0 0 0))
   (junction (at 36.83 116.84) (diameter 0.9144) (color 0 0 0 0))
@@
   (junction (at 195.58 27.94) (diameter 0.9144) (color 0 0 0 0))
   (junction (at 195.58 45.085) (diameter 0.9144) (color 0 0 0 0))
+  (no_connect (at 19.05 64.77))
   (no_connect (at 41.91 54.61))
   (no_connect (at 41.91 57.15))
@@
   (no_connect (at 192.405 40.005))
   (no_connect (at 192.405 42.545))
-  (wire (pts (xy 19.05 64.77) (xy 19.05 66.675))
+  (wire (pts (xy 26.67 64.77) (xy 26.67 69.215))
     (stroke (width 0) (type solid) (color 0 0 0 0))
   )
-  (wire (pts (xy 19.05 66.675) (xy 26.67 66.675))
-    (stroke (width 0) (type solid) (color 0 0 0 0))
-  )
-  (wire (pts (xy 26.67 64.77) (xy 26.67 66.675))
-    (stroke (width 0) (type solid) (color 0 0 0 0))
-  )
-  (wire (pts (xy 26.67 66.675) (xy 26.67 69.215))
-    (stroke (width 0) (type solid) (color 0 0 0 0))
-  )
