File: jlc_board/reptile-monitor.kicad_pcb (KiCad board)
At the start: 4 copper layers, 38.1 x 84.6 mm, 38 parts, among them IC1 ESP32-WROVER-E_M213EH6464PH3Q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, J1 UART, J2 AC_IN, J3 Conn_01x08, J7 LOAD1, J8 LOAD2, K1 ALDP105W, K2 ALDP105W, SW1 RST, SW2 BOOT, U1 NUD3105DMT1G, U3 AP2112K-3.3, Y1 32.768KHz 12.5p

Commit message: rev 2
Parts:
- removed C10, C7, C9: 0.1u, Capacitor_SMD:C_0603_1608Metric
- removed C8: 22u, Capacitor_SMD:C_0603_1608Metric
- removed IC1: ESP32-WROVER-E_M213EH6464PH3Q0_, SamacSys_Parts:ESP32WROVEREM213EH6464PH3Q0
- removed J7: LOAD1, reptile-monitor:Molex-43650-0215-0-0-MFG
- removed R12: 10k, Resistor_SMD:R_0603_1608Metric
- removed R13, R8: 100r, Resistor_SMD:R_0603_1608Metric
- removed REF1 (x2), REF2, REF3: MountingHole_2.2mm_M2, MountingHole:MountingHole_2.2mm_M2
- removed U3: AP2112K-3.3, SamacSys_Parts:SOIC127P600X170-8N
- removed svg2mod (x2): G***, svg2mod
- added C3: 0.1u, Capacitor_SMD:C_0603_1608Metric, F.Cu at (162.7, 112.4)
- added C4: 0.1u, Capacitor_SMD:C_0603_1608Metric, F.Cu at (161.2, 116.8)
- added C5: 22u, Capacitor_SMD:C_0603_1608Metric, F.Cu at (162.7, 116.8)
- added C6: 0.1u, Capacitor_SMD:C_0603_1608Metric, F.Cu at (137.4, 112.4)
- added FB1: 360 m, Capacitor_SMD:C_0805_2012Metric, F.Cu at (158.9, 84.6)
- added J4: LOAD1, reptile-monitor:Molex-43650-0215-0-0-MFG, F.Cu at (150.4, 39.2)
- added J5: LOAD2, reptile-monitor:Molex-43650-0215-0-0-MFG, F.Cu at (139.4, 39.1)
- added MD1: ESP32-WROVER-E, reptile-monitor:Espressif_Systems-ESP32-WROVER-0-0-MFG, F.Cu at (149.9, 109.9)
- added R2: 100r, Resistor_SMD:R_0603_1608Metric, F.Cu at (165.2, 95.6)
- added R3: 10k, Resistor_SMD:R_0603_1608Metric, F.Cu at (161.2, 112.4)
- added R4: 100r, Resistor_SMD:R_0603_1608Metric, F.Cu at (134.6, 95.6)
- added R5: 4.7k, Resistor_SMD:R_0603_1608Metric, F.Cu at (140.1, 91.2)
- added R6: 4.7k, Resistor_SMD:R_0603_1608Metric, F.Cu at (141.6, 91.2)
- added R7: 4.7k, Resistor_SMD:R_0603_1608Metric, F.Cu at (140.3, 86.1)
- added U2: NUD3105DMT1G, reptile-monitor:ON_Semi-318F-0-0-0, F.Cu at (145.4, 86.1)
- F1: value 39215000000 -> 39208000440
- J1: value UART -> 1-WIRE; footprint Connector_PinHeader_2.54mm:PinHeader_1x04_P2.54mm_Vertical -> Connector_JST:JST_SH_SM03B-SRSS-TB_1x03-1MP_P1.00mm_Horizontal
- J2: value AC_IN -> UART; footprint reptile-monitor:Molex-43650-0215-0-0-MFG -> Connector_PinHeader_2.54mm:PinHeader_1x04_P2.54mm_Vertical
- J3: value Conn_01x08 -> AC_IN; footprint Connector_PinHeader_2.54mm:PinHeader_2x06_P2.54mm_Vertical -> reptile-monitor:Molex-43650-0215-0-0-MFG
- J8: value LOAD2 -> I2C; footprint reptile-monitor:Molex-43650-0215-0-0-MFG -> Connector_JST:JST_SH_SM04B-SRSS-TB_1x04-1MP_P1.00mm_Horizontal
- U1: value NUD3105DMT1G -> AP2112M-3.3; footprint reptile-monitor:ON_Semi-318F-0-0-0 -> SamacSys_Parts:SOIC127P600X170-8N
- moved J2 66.0 mm to (135.1, 99.7)
- moved J3 57.3 mm to (161.3, 39.1), turned to 0 degrees
- moved J8 49.9 mm to (134.2, 88.8), turned to -90 degrees
- moved D2 30.1 mm to (136.1, 95.6)
- moved R1 26.2 mm to (164.8, 86.0), turned to 180 degrees
- moved J1 20.2 mm to (134.2, 79.6), turned to -90 degrees
- moved U1 12.2 mm to (165.1, 90.4), turned to 90 degrees
- moved D1 6.75 mm to (166.8, 95.6)
- moved WESLEY 5.97 mm to (144.4, 83.6)
- moved SW1 1.40 mm to (165.6, 112.3)
- moved SW2 1.27 mm to (135.1, 112.3)
- moved CL1 0.76 mm to (164.3, 108.3)
- moved CL2 0.76 mm to (164.3, 106.3)
- moved Y1 0.58 mm to (161.6, 107.3)
Connections:
- C1 pad 1: +5V -> Net-(C1-Pad1)
- D1 pad 1: /IO13 -> GND
- D2 pad 1: GND -> LED
- J1 pad 1: +3V3 -> GND
- J1 pad 2: /RXD0 -> /IO27
- J1 pad 3: /TXD0 -> +3V3
- J2 pad 1: /AC_L -> +3V3
- J2 pad 2: /AC_N -> RXD0
- J3 pad 1: /IO18 -> /AC_L
- J3 pad 2: /IO19 -> /AC_N
- J8 pad 1: /LOAD2 -> +3V3
- J8 pad 2: /AC_N -> /IO26
- R1 pad 1: /EN -> /PWR_EN
- R1 pad 2: Net-(C9-Pad1) -> Net-(C1-Pad1)
- SW1 pad 1: Net-(C9-Pad1) -> Net-(C3-Pad1)
- U1 pad 1: GND -> +3V3
- U1 pad 2: /IO14 -> (no net)
- U1 pad 3: /RLY2 -> (no net)
- U1 pad 4: GND -> (no net)
- U1 pad 5: /IO12 -> /PWR_EN
- U1 pad 6: /RLY1 -> GND
Routing:
- net /IO36: track 34.7 -> 0.00 mm
- net /IO22: track 31.8 -> 0.00 mm
- net /IO23: track 29.9 -> 0.00 mm
- net /IO39: track 29.6 -> 0.00 mm
- net /IO19: track 26.6 -> 0.00 mm
- net /IO21: track 25.2 -> 0.00 mm
- net SCLK: track 0.00 -> 23.9 mm
- net MISO: track 0.00 -> 21.9 mm
- net /IO5: track 21.9 -> 0.00 mm
- net /IO18: track 21.8 -> 0.00 mm
- net /IO14: track 20.4 -> 0.00 mm
- net /IO12: track 17.4 -> 0.00 mm
- net +5V: track 48.1 -> 32.1 mm
- net RXD0: track 0.00 -> 14.1 mm
- net /RXD0: track 14.1 -> 0.00 mm
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- added copper zone on F.Cu, net +3V3
- added copper zone on F.Cu, net +5V
- added copper zone on F.Cu, net Net-(C1-Pad1)
Other:
- board text added: "JLCJLCJLCJLC"
- board text added: "Mike Pleimann"
- board text added: "Reptile Monitor"
- board text added: "Rev. 2 May 2021"
- board text removed: "15"
- board text removed: "18"
- board text removed: "19"
- board text removed: "21"
- board text removed: "22"
- board text removed: "23"
- board text removed: "25"
- board text removed: "26"
- board text removed: "27"
- board text removed: "36"
- board text removed: "39"
- board text removed: "5"
- board text removed: "Rev 2 April 2021"

Commit message: Rev2 - Waffle & Wesley
Parts:
- added J6: I/O, Connector_PinHeader_1.27mm:PinHeader_2x05_P1.27mm_Vertical_SMD, F.Cu at (135.3, 117.7)
- added REF1: MountingHole_2.2mm_M2_ISO7380, MountingHole:MountingHole_2.2mm_M2_ISO7380, F.Cu at (137.2, 53.3)
- added REF1: MountingHole_2.2mm_M2_ISO7380, MountingHole:MountingHole_2.2mm_M2_ISO7380, F.Cu at (104.1, 132.8)
- added REF1: MountingHole_2.2mm_M2_ISO7380, MountingHole:MountingHole_2.2mm_M2_ISO7380, F.Cu at (104.1, 53.3)
- added REF1: MountingHole_2.2mm_M2_ISO7380, MountingHole:MountingHole_2.2mm_M2_ISO7380, F.Cu at (137.2, 132.8)
- C1, C2: footprint Capacitor_SMD:C_0805_2012Metric -> Capacitor_SMD:C_0603_1608Metric
- FB1: footprint Capacitor_SMD:C_0805_2012Metric -> Inductor_SMD:L_0805_2012Metric
- J3: footprint reptile-monitor:Molex-43650-0215-0-0-MFG -> SamacSys_Parts:128340212
- J4: value LOAD1 -> LOAD_1; footprint reptile-monitor:Molex-43650-0215-0-0-MFG -> SamacSys_Parts:128340212
- J5: value LOAD2 -> LOAD_2; footprint reptile-monitor:Molex-43650-0215-0-0-MFG -> SamacSys_Parts:128340212
- SW1: value RST -> RESET
- moved RV1 48.2 mm to (106.9, 57.9), turned to -90 degrees
- moved J3 39.1 mm to (126.6, 57.1), turned to 180 degrees
- moved R6 35.6 mm to (110.4, 108.2), turned to -90 degrees
- moved J4 35.3 mm to (120.0, 57.1), turned to 180 degrees
- moved CL2 34.6 mm to (134.6, 124.0)
- moved Y1 34.5 mm to (131.8, 124.7)
- moved CL1 34.4 mm to (134.6, 125.5)
- moved SW1 33.9 mm to (135.9, 128.5)
- moved C6 33.9 mm to (107.7, 128.7)
- moved SW2 33.9 mm to (105.4, 128.5)
- moved F1 33.9 mm to (137.3, 62.1)
- moved C3 33.8 mm to (133.0, 128.5)
- moved R3 33.8 mm to (131.4, 128.5)
- moved C4 33.8 mm to (131.4, 132.9)
- moved C5 33.8 mm to (133.0, 132.9)
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Connections:
- net /IO0 renamed BOOT
- F1 pad 1: /AC_L -> /FUSED_AC_L
- F1 pad 2: /FUSED_AC_L -> /AC_L
- J1 pad 2: /IO27 -> 1-WIRE
- J4 pad 1: /LOAD1 -> /AC_N
- J4 pad 2: /AC_N -> /LOAD1
- J5 pad 1: /LOAD2 -> /AC_N
- J5 pad 2: /AC_N -> /LOAD2
- J8 pad 2: /IO26 -> SDA
- J8 pad 3: /IO25 -> SCL
- MD1 pad 10: /IO25 -> IO25
- MD1 pad 11: /IO26 -> IO26
- MD1 pad 12: /IO27 -> IO27
- MD1 pad 13: SCLK -> SCK
- MD1 pad 14: MISO -> SDI
- MD1 pad 16: (no net) -> SDO
- MD1 pad 23: (no net) -> CS0
- MD1 pad 26: (no net) -> SCL
- MD1 pad 29: (no net) -> SDA
- MD1 pad 30: (no net) -> 1-WIRE
- MD1 pad 31: (no net) -> L1
- MD1 pad 33: (no net) -> L2
- R5 pad 2: /IO25 -> SDA
- R6 pad 2: /IO26 -> SCL
- R7 pad 2: /IO27 -> 1-WIRE
- U2 pad 2: SCLK -> L1
- U2 pad 5: MISO -> L2
Routing:
- net L2: track 0.00 -> 37.3 mm
- net 1-WIRE: track 0.00 -> 35.5 mm
- net L1: track 0.00 -> 34.0 mm
- net /IO27: track 33.9 -> 0.00 mm
- net /IO25: track 28.7 -> 0.00 mm
- net /IO26: track 28.6 -> 0.00 mm
- net CS0: track 0.00 -> 27.1 mm, vias 0 -> 2
- net SDA: track 0.00 -> 26.9 mm
- net SCLK: track 23.9 -> 0.00 mm
- net MISO: track 21.9 -> 0.00 mm
- net SCL: track 0.00 -> 20.1 mm
- net IO25: track 0.00 -> 10.3 mm
- net IO26: track 0.00 -> 8.58 mm
- net SCK: track 0.00 -> 8.43 mm
- net IO27: track 0.00 -> 7.58 mm
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Other:
- outline, holes or cut-outs redrawn
- board text added: "25"
- board text added: "26"
- board text added: "27"
- board text added: "CS"
- board text added: "SCK"
- board text added: "SDI"
- board text added: "SDO"

Commit message: Revision 3
Parts:
- removed CL1, CL2: 20p, Capacitor_SMD:C_0603_1608Metric
- removed Y1: 32.768KHz 12.5p, reptile-monitor:Crystal_SMD_3215-2Pin_3.2x1.5mm
- added C7: 100n, Capacitor_SMD:C_0603_1608Metric, F.Cu at (133.0, 125.5)
- added D3: Schottky, Diode_SMD:D_SOD-523, F.Cu at (120.1, 101.2)
- added svg2mod: G***, svg2mod, B.Cu at (132.1, 91.4)
- C3, C6: value 0.1u -> 100n
- C4: value 0.1u -> 22u
- C5: value 22u -> 100n
- D1: value LED -> RED
- D2: value LED -> BLUE
- FB1: footprint Inductor_SMD:L_0805_2012Metric -> Inductor_SMD:L_0603_1608Metric_Pad1.05x0.95mm_HandSolder
- R2, R4: value 100r -> 10k
- R5, R6, R7: value 4.7k -> 10k
- SW1, SW2: footprint reptile-monitor:Omron-B3U-1000P-MFG -> reptile-monitor:CK-KMR221GLFS-MFG
- moved J2 25.2 mm to (127.8, 104.3), turned to -90 degrees
- moved U2 5.85 mm to (116.0, 102.2)
- moved R4 2.94 mm to (107.8, 111.8)
- moved C6 2.19 mm to (107.3, 126.5)
- moved SW2 1.44 mm to (104.4, 127.5)
- moved SW1 1.44 mm to (136.9, 127.5), turned to 90 degrees
- moved WESLEY 0.94 mm to (114.2, 100.5)
- moved R5 0.76 mm to (112.6, 108.2)
- moved R6 0.76 mm to (111.1, 108.2)
- moved R7 0.64 mm to (114.2, 108.2)
- moved D2 0.07 mm to (106.4, 111.8)
Connections:
- C3 pad 1: Net-(C3-Pad1) -> /EN
- D2 pad 1: LED -> GND
- J2 pad 1: +3V3 -> GND
- J2 pad 2: RXD0 -> TXD0
- J2 pad 3: TXD0 -> RXD0
- J2 pad 4: GND -> Net-(D3-Pad2)
- J6 pad 1: +3V3 -> IO26
- J6 pad 3: IO27 -> IO25
- J6 pad 5: IO26 -> IO35
- J6 pad 7: IO25 -> IO34
- MD1 pad 12: IO27 -> CS0
- MD1 pad 23: CS0 -> /LED
- MD1 pad 24: LED -> (no net)
- MD1 pad 6: (no net) -> IO34
- MD1 pad 7: (no net) -> IO35
- MD1 pad 8: Net-(CL1-Pad1) -> (no net)
- MD1 pad 9: Net-(CL2-Pad1) -> (no net)
- R3 pad 2: Net-(C3-Pad1) -> +3V3
- R4 pad 2: GND -> /LED
- SW1 pad 1: Net-(C3-Pad1) -> /EN
- SW1 pad 2: GND -> /EN
- SW2 pad 2: GND -> BOOT
Routing:
- net +5V: track 32.1 -> 0.00 mm
- net TXD0: track 12.9 -> 32.8 mm
- net RXD0: track 14.1 -> 30.7 mm
- net CS0: track 27.1 -> 11.3 mm, vias 2 -> 0
- net IO34: track 0.00 -> 12.2 mm
- net /EN: track 4.04 -> 15.1 mm
- net IO35: track 0.00 -> 9.97 mm
- net BOOT: track 27.6 -> 18.1 mm
- net L2: track 37.3 -> 29.4 mm
- net IO27: track 7.58 -> 0.00 mm
- net LED: track 6.74 -> 0.00 mm
- net /RLY1: track 11.1 -> 17.2 mm
- net /RLY2: track 15.9 -> 21.8 mm
- net L1: track 34.0 -> 28.2 mm
- net Net-(CL2-Pad1): track 5.49 -> 0.00 mm
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Other:
- board text added: "34"
- board text added: "35"
- board text added: "5V"
- board text added: "Rev. 3 June 2021"
- board text added: "[3V3]"
- board text removed: "27"
- board text removed: "Reptile Monitor"
- board text removed: "Rev. 2 May 2021"
