File: jlc_board/_autosave-reptile-monitor-rounded.kicad_pcb (KiCad board)
At the start: 4 copper layers, 38.1 x 38.1 mm, 29 parts, among them J1 AudioJack4_SwitchR1, J2 AudioJack4_SwitchR1, J3 PWR CONN, J4 UART, J6 18-Lead FPC 0.5 mm - Vertical, Q1 Q_NPN_BEC, SW1 RESET, U1 AP2112M-3.3

Commit message: tt-relay
Parts:
- removed R4: 1k, reptile-monitor:R_0603_1608Metric
- D2: value 32 -> WS2812B; footprint reptile-monitor:LED_0603_1608Metric -> reptile-monitor:LED_WS2812B_PLCC4_5.0x5.0mm_P3.2mm
- U1: footprint Package_TO_SOT_SMD:SOT-223 -> reptile-monitor:SOIC127P600X170-8N
- moved Q1 11.7 mm to (129.7, 108.0)
- moved D2 10.4 mm to (120.7, 103.0), turned to 0 degrees
- moved R5 8.44 mm to (129.7, 105.1), turned to 0 degrees
- moved D4 1.78 mm to (121.4, 96.5)
- moved D5 1.78 mm to (123.3, 96.5)
- moved C1 1.78 mm to (119.1, 96.2)
- moved R1 1.78 mm to (117.6, 96.2)
- moved U1 1.51 mm to (119.5, 90.8)
Connections:
- D2 pad 1: GND -> +3V3
- D2 pad 2: Net-(D2-Pad2) -> unconnected-(D2-Pad2)
- MD1 pad 8: /LED -> LED
Routing:
- net LED: track 0.00 -> 14.9 mm
- net GND: track 31.7 -> 35.0 mm, vias 26 -> 29
- net Net-(D3-Pad2): track 9.34 -> 6.50 mm
- net TXD0: track 35.9 -> 33.8 mm
- net +5V: track 6.35 -> 8.29 mm
- net Net-(J4-Pad3): track 28.0 -> 29.8 mm
- net BUZZER: track 18.9 -> 20.7 mm
- net /PWR_EN: track 0.00 -> 1.68 mm
- net +3V3: track 14.9 -> 16.4 mm, vias 9 -> 13
- net EN: track 72.8 -> 71.4 mm
- net Net-(J3-Pad2): track 23.1 -> 22.0 mm
- net BOOT: track 9.83 -> 8.82 mm
Other:
- board text added: "Rev. 5 - April 2022"
- board text removed: "Rev. 5 Feb 2022"
